File: hardware/design/Power.sch (KiCad schematic (older format))
At the start: 11 parts, among them U5 NCP1117ST50T3G, U6 LP2992AIM5-3.3

Commit message: Six-phase power stage.
Parts:
- renumbered R10 to R3vi1, U5 to Ureg1, U6 to Ureg2
Changed lines of the file:
@@
 $Descr A4 11693 8268
 encoding utf-8
-Sheet 5 6
+Sheet 5 12
 Title "DrChibi"
 Date "25 Aug 2014"
@@
 AB D8 39 0B 59 91 9E DF A8 2A 5B EE 54 3A FD 71 ED 71 2F 29 C3 82 EC 80 87 06 6E C3 98 10 30 3B
 62 9A BB 2D 03 B8 C4 64 FC B5 26 AC 13 9B D1 39 40 41 C1 D6 78 4C 84 BF 94 F0 6F E1 BF 96 F0 0F
-FF 77 E2 FF 1F 0F 43 55 32 21 1C 08 16 00 00 00 00 49 45 4E 44 AE 42 60 82 1B
+FF 77 E2 FF 1F 0F 43 55 32 21 1C 08 16 00 00 00 00 49 45 4E 44 AE 42 60 82 6C
 EndData
 $EndBitmap
@@
 	5900 1150 5400 1150
 $Comp
-L GNDPWR #PWR42
+L GNDPWR #PWR43
 U 1 1 55E7501A
 P 6300 1750
-F 0 "#PWR42" H 6300 1550 50  0001 C CNN
+F 0 "#PWR43" H 6300 1550 50  0001 C CNN
 F 1 "GNDPWR" H 6300 1620 50  0000 C CNN
 F 2 "" H 6300 1700 60  0000 C CNN
@@
 $EndComp
 $Comp
-L GNDPWR #PWR47
+L GNDPWR #PWR48
 U 1 1 55E7507A
 P 10400 1650
-F 0 "#PWR47" H 10400 1450 50  0001 C CNN
+F 0 "#PWR48" H 10400 1450 50  0001 C CNN
 F 1 "GNDPWR" H 10400 1520 50  0000 C CNN
 F 2 "" H 10400 1600 60  0000 C CNN
@@
 $EndComp
 $Comp
-L +24V #PWR46
+L +24V #PWR47
 U 1 1 56A6E18F
 P 10400 750
-F 0 "#PWR46" H 10400 600 50  0001 C CNN
+F 0 "#PWR47" H 10400 600 50  0001 C CNN
 F 1 "+24V" H 10418 924 50  0000 C CNN
 F 2 "" H 10400 750 50  0000 C CNN
@@
 $EndComp
 $Comp
-L +24V #PWR41
+L +24V #PWR42
 U 1 1 56A6E22C
 P 5400 1150
-F 0 "#PWR41" H 5400 1000 50  0001 C CNN
+F 0 "#PWR42" H 5400 1000 50  0001 C CNN
 F 1 "+24V" V 5418 1277 50  0000 L CNN
 F 2 "" H 5400 1150 50  0000 C CNN
@@
 $EndComp
 $Comp
-L NCP1117ST50T3G U5
+L NCP1117ST50T3G Ureg1
 U 1 1 56A901A9
 P 6300 1200
-F 0 "U5" H 6300 1610 50  0000 C CNN
+F 0 "Ureg1" H 6300 1610 50  0000 C CNN
 F 1 "NCP1117ST50T3G" H 6300 1518 50  0000 C CNN
 F 2 "TO_SOT_Packages_SMD:SOT-223" H 6300 1426 50  0000 C CNN
@@
 $EndComp
 $Comp
-L +5V #PWR44
+L +5V #PWR45
 U 1 1 56A9035F
 P 7250 1050
-F 0 "#PWR44" H 7250 900 50  0001 C CNN
+F 0 "#PWR45" H 7250 900 50  0001 C CNN
 F 1 "+5V" H 7268 1224 50  0000 C CNN
 F 2 "" H 7250 1050 50  0000 C CNN
@@
 $EndComp
 $Comp
-L GND #PWR43
+L GND #PWR44
 U 1 1 56A90F82
 P 6350 3850
-F 0 "#PWR43" H 6350 3600 50  0001 C CNN
+F 0 "#PWR44" H 6350 3600 50  0001 C CNN
 F 1 "GND" H 6358 3676 50  0000 C CNN
 F 2 "" H 6350 3850 50  0000 C CNN
@@
 $EndComp
 $Comp
-L +5V #PWR40
+L +5V #PWR41
 U 1 1 56A9100E
 P 5200 3400
-F 0 "#PWR40" H 5200 3250 50  0001 C CNN
+F 0 "#PWR41" H 5200 3250 50  0001 C CNN
 F 1 "+5V" H 5218 3574 50  0000 C CNN
 F 2 "" H 5200 3400 50  0000 C CNN
@@
 $EndComp
 $Comp
-L +3.3V #PWR45
+L +3.3V #PWR46
 U 1 1 56A9147A
 P 7250 3250
-F 0 "#PWR45" H 7250 3100 50  0001 C CNN
+F 0 "#PWR46" H 7250 3100 50  0001 C CNN
 F 1 "+3.3V" H 7268 3424 50  0000 C CNN
 F 2 "" H 7250 3250 50  0000 C CNN
@@
 Connection ~ 7250 3400
 $Comp
-L LP2992AIM5-3.3 U6
+L LP2992AIM5-3.3 Ureg2
 U 1 1 56A909DA
 P 6350 3450
-F 0 "U6" H 6350 3768 50  0000 C CNN
+F 0 "Ureg2" H 6350 3768 50  0000 C CNN
 F 1 "LP2992AIM5-3.3" H 6350 3676 50  0000 C CNN
 F 2 "TO_SOT_Packages_SMD:SOT-23-5" H 6350 3676 50  0001 C CIN
@@
 3.3V regulator\nfor the logic
 $Comp
-L R R10
+L R R3vi1
 U 1 1 56A53CCD
 P 5350 3400
-F 0 "R10" V 5142 3400 50  0000 C CNN
+F 0 "R3vi1" V 5142 3400 50  0000 C CNN
 F 1 "2R7" V 5234 3400 50  0000 C CNN
 F 2 "Resistors_SMD:R_1206" V 5280 3400 50  0001 C CNN

Commit message: Changed pin for LED3
Parts:
- Cpwr1: Comment (none) -> X7R, e.g. GRM32ER7YA106KA12L
Other:
- note added: "Consider RC-line-filtering here as well."
Changed lines of the file:
@@
 F 2 "Capacitors_SMD:C_1206" H 10400 1300 60  0001 C CNN
 F 3 "" H 10400 1300 60  0001 C CNN
+F 4 "X7R, e.g. GRM32ER7YA106KA12L" V 10400 1300 60  0001 C CNN "Comment"
 	1    10400 1300
 	-1   0    0    1
@@
 AB D8 39 0B 59 91 9E DF A8 2A 5B EE 54 3A FD 71 ED 71 2F 29 C3 82 EC 80 87 06 6E C3 98 10 30 3B
 62 9A BB 2D 03 B8 C4 64 FC B5 26 AC 13 9B D1 39 40 41 C1 D6 78 4C 84 BF 94 F0 6F E1 BF 96 F0 0F
-FF 77 E2 FF 1F 0F 43 55 32 21 1C 08 16 00 00 00 00 49 45 4E 44 AE 42 60 82 09
+FF 77 E2 FF 1F 0F 43 55 32 21 1C 08 16 00 00 00 00 49 45 4E 44 AE 42 60 82 48
 EndData
 $EndBitmap
@@
 Text Notes 5200 3650 0    40   ~ 0
 Line\nfilter\nRC
+Text Notes 5450 2100 0    60   ~ 0
+Consider RC-line-filtering here as well.
 $EndSCHEMATC
