File: hardware/design/half_bridge_insd.sch (KiCad schematic (older format))
At the start: 13 parts

Commit message: Six-phase power stage.
Parts:
- added Csens1: 0.47u, Capacitors_SMD:C_0603, symbol C
- Ccfilt1: footprint Capacitors_SMD:C_0603_HandSoldering -> Capacitors_SMD:C_0402
- Rcfilt1, Rlsens1: footprint Capacitors_SMD:C_0603_HandSoldering -> Resistors_SMD:R_0402
Connections:
- net +3V3: now also Csens1.1
- net GND: now also Csens1.2
- no-connect marks 0 -> 2
Other:
- note added: "Csens is the bypass capacitor for ACS711"
- note added: "SENSV = Rlsens / (Rlsens+Rhsens)\nMust be below 4V to protect the input pin of STM32F4.\nIs 3.8V for Rl=2k2 and Rh=10k\n\nNote:\nThink about placing Rlsens close to the controller and\nRhsens at the pad. Having load at the wire would make\nit less susceptible to noise."
- note removed: "SENSV = Rlsens / (Rlsens+Rhsens)\nMust be below 4V to protect the input pin of STM32F4.\nIs 3.8V for Rl=2k2 and Rh=10k"

Commit message: TODO: Find appropriate routing to CPU
Changed lines of the file:
@@
 AR Path="/56BA2E2B/55DF8D4F" Ref="Cboot5"  Part="1"
 AR Path="/56BA5F82/55DF8D4F" Ref="Cboot6"  Part="1"
-F 0 "Cboot6" V 6647 3700 50  0000 C CNN
+F 0 "Cboot1" V 6647 3700 50  0000 C CNN
 F 1 "0.47uF" V 6739 3700 50  0000 C CNN
 F 2 "Capacitors_SMD:C_0603_HandSoldering" H 6938 3550 30  0001 C CNN
@@
 AR Path="/56BA2E2B/55DF8D84" Ref="CDrGate5"  Part="1"
 AR Path="/56BA5F82/55DF8D84" Ref="CDrGate6"  Part="1"
-F 0 "CDrGate6" H 5065 2946 50  0000 L CNN
+F 0 "CDrGate1" H 5065 2946 50  0000 L CNN
 F 1 "0.47uF" H 5065 2854 50  0000 L CNN
 F 2 "Capacitors_SMD:C_0603_HandSoldering" H 4988 2750 30  0001 C CNN
@@
 AR Path="/56BA2E2B/56984538" Ref="Usens5"  Part="1"
 AR Path="/56BA5F82/56984538" Ref="Usens6"  Part="1"
-F 0 "Usens6" V 7797 2922 60  0000 R CNN
+F 0 "Usens1" V 7797 2922 60  0000 R CNN
 F 1 "ACS711" V 7903 2922 60  0000 R CNN
 F 2 "Allegro:QFN-12-1EX_3x3mm_Pitch0.5mm" V 7956 2922 60  0001 R CNN
@@
 AR Path="/56BA2E2B/56A19C85" Ref="UDrmos5"  Part="1"
 AR Path="/56BA5F82/56A19C85" Ref="UDrmos6"  Part="1"
-F 0 "UDrmos6" H 5650 5071 50  0000 C CNN
+F 0 "UDrmos1" H 5650 5071 50  0000 C CNN
 F 1 "DrMOS_SiC632A" H 5650 4979 50  0000 C CNN
 F 2 "DrMOS:MLP55-31L" H 5650 4887 50  0000 C CNN
@@
 AR Path="/56BA2E2B/56A2AE4F" Ref="#PWR94"  Part="1"
 AR Path="/56BA5F82/56A2AE4F" Ref="#PWR107"  Part="1"
-F 0 "#PWR107" H 5750 4850 50  0001 C CNN
+F 0 "#PWR34" H 5750 4850 50  0001 C CNN
 F 1 "GNDPWR" H 5750 4900 50  0000 C CNN
 F 2 "" H 5750 5000 50  0000 C CNN
@@
 AR Path="/56BA2E2B/56A2B769" Ref="#PWR91"  Part="1"
 AR Path="/56BA5F82/56A2B769" Ref="#PWR104"  Part="1"
-F 0 "#PWR104" H 5200 4750 50  0001 C CNN
+F 0 "#PWR31" H 5200 4750 50  0001 C CNN
 F 1 "GND" H 5208 4826 50  0000 C CNN
 F 2 "" H 5200 5000 50  0000 C CNN
@@
 AR Path="/56BA2E2B/56A2BBEE" Ref="#PWR90"  Part="1"
 AR Path="/56BA5F82/56A2BBEE" Ref="#PWR103"  Part="1"
-F 0 "#PWR103" H 4950 3000 50  0001 C CNN
+F 0 "#PWR30" H 4950 3000 50  0001 C CNN
 F 1 "GNDPWR" H 4957 3275 50  0000 C CNN
 F 2 "" H 4950 3150 50  0000 C CNN
@@
 AR Path="/56BA2E2B/56A2CDC4" Ref="CDrLogic5"  Part="1"
 AR Path="/56BA5F82/56A2CDC4" Ref="CDrLogic6"  Part="1"
-F 0 "CDrLogic6" H 4415 3446 50  0000 L CNN
+F 0 "CDrLogic1" H 4415 3446 50  0000 L CNN
 F 1 "2.2uF" H 4415 3354 50  0000 L CNN
 F 2 "Capacitors_SMD:C_0603" H 4338 3250 30  0001 C CNN
@@
 AR Path="/56BA2E2B/56A2CDEC" Ref="#PWR89"  Part="1"
 AR Path="/56BA5F82/56A2CDEC" Ref="#PWR102"  Part="1"
-F 0 "#PWR102" H 4300 3300 50  0001 C CNN
+F 0 "#PWR29" H 4300 3300 50  0001 C CNN
 F 1 "GND" H 4308 3376 50  0000 C CNN
 F 2 "" H 4300 3550 50  0000 C CNN
@@
 AR Path="/56BA2E2B/56A2CF9B" Ref="#PWR88"  Part="1"
 AR Path="/56BA5F82/56A2CF9B" Ref="#PWR101"  Part="1"
-F 0 "#PWR101" H 4300 2500 50  0001 C CNN
+F 0 "#PWR28" H 4300 2500 50  0001 C CNN
 F 1 "+5V" H 4318 2824 50  0000 C CNN
 F 2 "" H 4300 2650 50  0000 C CNN
@@
 AR Path="/56BA2E2B/56A2D0BC" Ref="RDrLogic5"  Part="1"
 AR Path="/56BA5F82/56A2D0BC" Ref="RDrLogic6"  Part="1"
-F 0 "RDrLogic6" H 4370 2946 50  0000 L CNN
+F 0 "RDrLogic1" H 4370 2946 50  0000 L CNN
 F 1 "R" H 4370 2854 50  0000 L CNN
 F 2 "Resistors_SMD:R_0603" V 4230 2900 50  0001 C CNN
@@
 AR Path="/56BA2E2B/56A2EFF6" Ref="#PWR100"  Part="1"
 AR Path="/56BA5F82/56A2EFF6" Ref="#PWR113"  Part="1"
-F 0 "#PWR113" H 8550 2800 50  0001 C CNN
+F 0 "#PWR40" H 8550 2800 50  0001 C CNN
 F 1 "GND" H 8558 2876 50  0000 C CNN
 F 2 "" H 8550 3050 50  0000 C CNN
@@
 AR Path="/56BA2E2B/56A2FD69" Ref="Rhsens5"  Part="1"
 AR Path="/56BA5F82/56A2FD69" Ref="Rhsens6"  Part="1"
-F 0 "Rhsens6" H 7520 4346 50  0000 L CNN
+F 0 "Rhsens1" H 7520 4346 50  0000 L CNN
 F 1 "10k" H 7520 4254 50  0000 L CNN
 F 2 "Capacitors_SMD:C_0603_HandSoldering" V 7380 4300 50  0001 C CNN
@@
 AR Path="/56BA2E2B/56A2FEAC" Ref="Rlsens5"  Part="1"
 AR Path="/56BA5F82/56A2FEAC" Ref="Rlsens6"  Part="1"
-F 0 "Rlsens6" H 7520 4746 50  0000 L CNN
+F 0 "Rlsens1" H 7520 4746 50  0000 L CNN
 F 1 "2k2" H 7520 4654 50  0000 L CNN
 F 2 "Resistors_SMD:R_0402" V 7380 4700 50  0001 C CNN
@@
 AR Path="/56BA2E2B/56A30067" Ref="#PWR99"  Part="1"
 AR Path="/56BA5F82/56A30067" Ref="#PWR112"  Part="1"
-F 0 "#PWR112" H 7450 4700 50  0001 C CNN
+F 0 "#PWR39" H 7450 4700 50  0001 C CNN
 F 1 "GND" H 7458 4776 50  0000 C CNN
 F 2 "" H 7450 4950 50  0000 C CNN
@@
 AR Path="/56BA2E2B/56A31D68" Ref="#PWR95"  Part="1"
 AR Path="/56BA5F82/56A31D68" Ref="#PWR108"  Part="1"
-F 0 "#PWR108" H 6050 2850 50  0001 C CNN
+F 0 "#PWR35" H 6050 2850 50  0001 C CNN
 F 1 "+24V" H 6068 3174 50  0000 C CNN
 F 2 "" H 6050 3000 50  0000 C CNN
@@
 AR Path="/56BA2E2B/56A32138" Ref="#PWR98"  Part="1"
 AR Path="/56BA5F82/56A32138" Ref="#PWR111"  Part="1"
-F 0 "#PWR111" H 7350 2500 50  0001 C CNN
+F 0 "#PWR38" H 7350 2500 50  0001 C CNN
 F 1 "+3.3V" H 7368 2824 50  0000 C CNN
 F 2 "" H 7350 2650 50  0000 C CNN
@@
 AR Path="/56BA2E2B/56A3225A" Ref="Rcfilt5"  Part="1"
 AR Path="/56BA5F82/56A3225A" Ref="Rcfilt6"  Part="1"
-F 0 "Rcfilt6" H 8420 2846 50  0000 L CNN
+F 0 "Rcfilt1" H 8420 2846 50  0000 L CNN
 F 1 "R" H 8420 2754 50  0000 L CNN
 F 2 "Resistors_SMD:R_0402" V 8280 2800 50  0001 C CNN
@@
 AR Path="/56BA2E2B/56A3233B" Ref="Ccfilt5"  Part="1"
 AR Path="/56BA5F82/56A3233B" Ref="Ccfilt6"  Part="1"
-F 0 "Ccfilt6" H 8165 2846 50  0000 L CNN
+F 0 "Ccfilt1" H 8165 2846 50  0000 L CNN
 F 1 "C" H 8165 2754 50  0000 L CNN
 F 2 "Capacitors_SMD:C_0402" H 8088 2650 50  0001 C CNN
@@
 AR Path="/56BA2E2B/56A69AD2" Ref="#PWR92"  Part="1"
 AR Path="/56BA5F82/56A69AD2" Ref="#PWR105"  Part="1"
-F 0 "#PWR105" H 5750 800 50  0001 C CNN
+F 0 "#PWR32" H 5750 800 50  0001 C CNN
 F 1 "+24V" H 5768 1124 50  0000 C CNN
 F 2 "" H 5750 950 50  0000 C CNN
@@
 AR Path="/56BA2E2B/56A69B0E" Ref="CDrHV5"  Part="1"
 AR Path="/56BA5F82/56A69B0E" Ref="CDrHV6"  Part="1"
-F 0 "CDrHV6" H 5865 1246 50  0000 L CNN
+F 0 "CDrHV1" H 5865 1246 50  0000 L CNN
 F 1 "10u" H 5865 1154 50  0000 L CNN
 F 2 "Capacitors_SMD:C_1206" H 5788 1050 50  0001 C CNN
@@
 AR Path="/56BA2E2B/56A69BA7" Ref="#PWR93"  Part="1"
 AR Path="/56BA5F82/56A69BA7" Ref="#PWR106"  Part="1"
-F 0 "#PWR106" H 5750 1300 50  0001 C CNN
+F 0 "#PWR33" H 5750 1300 50  0001 C CNN
 F 1 "GNDPWR" H 5757 1575 50  0000 C CNN
 F 2 "" H 5750 1450 50  0000 C CNN
@@
 AR Path="/56BA2E2B/56AF6D20" Ref="CDrHVs5"  Part="1"
 AR Path="/56BA5F82/56AF6D20" Ref="CDrHVs6"  Part="1"
-F 0 "CDrHVs6" H 5315 1246 50  0000 L CNN
+F 0 "CDrHVs1" H 5315 1246 50  0000 L CNN
 F 1 "0.47u" H 5315 1154 50  0000 L CNN
 F 2 "Capacitors_SMD:C_0603" H 5315 1108 50  0001 L CNN
@@
 AR Path="/56BA2E2B/56B30AD6" Ref="PMotor5"  Part="1"
 AR Path="/56BA5F82/56B30AD6" Ref="PMotor6"  Part="1"
-F 0 "PMotor6" H 9177 4106 60  0000 L CNN
+F 0 "PMotor1" H 9177 4106 60  0000 L CNN
 F 1 "PAD_SMD" H 9177 4000 60  0000 L CNN
 F 2 "CRF1:1PAD_4x5mm" H 9177 3894 60  0000 L CNN
@@
 AR Path="/56BA2E2B/56B897AB" Ref="Csens5"  Part="1"
 AR Path="/56BA5F82/56B897AB" Ref="Csens6"  Part="1"
-F 0 "Csens6" H 6965 2142 50  0000 L CNN
+F 0 "Csens1" H 6965 2142 50  0000 L CNN
 F 1 "0.47u" H 6965 2050 50  0000 L CNN
 F 2 "Capacitors_SMD:C_0603" H 6965 1958 50  0000 L CNN
@@
 AR Path="/56BA2E2B/56B89931" Ref="#PWR97"  Part="1"
 AR Path="/56BA5F82/56B89931" Ref="#PWR110"  Part="1"
-F 0 "#PWR110" H 6850 1950 50  0001 C CNN
+F 0 "#PWR37" H 6850 1950 50  0001 C CNN
 F 1 "GND" H 6858 2026 50  0000 C CNN
 F 2 "" H 6850 2200 50  0000 C CNN
@@
 AR Path="/56BA2E2B/56B89961" Ref="#PWR96"  Part="1"
 AR Path="/56BA5F82/56B89961" Ref="#PWR109"  Part="1"
-F 0 "#PWR109" H 6850 1750 50  0001 C CNN
+F 0 "#PWR36" H 6850 1750 50  0001 C CNN
 F 1 "+3.3V" H 6868 2074 50  0000 C CNN
 F 2 "" H 6850 1900 50  0000 C CNN

Commit message: Changed pin for LED3
Changed lines of the file:
@@
 AR Path="/56BA2E2B/55DF8D4F" Ref="Cboot5"  Part="1"
 AR Path="/56BA5F82/55DF8D4F" Ref="Cboot6"  Part="1"
-F 0 "Cboot6" V 6647 3700 50  0000 C CNN
+F 0 "Cboot1" V 6647 3700 50  0000 C CNN
 F 1 "0.47uF" V 6739 3700 50  0000 C CNN
 F 2 "Capacitors_SMD:C_0603_HandSoldering" H 6938 3550 30  0001 C CNN
@@
 AR Path="/56BA2E2B/55DF8D84" Ref="CDrGate5"  Part="1"
 AR Path="/56BA5F82/55DF8D84" Ref="CDrGate6"  Part="1"
-F 0 "CDrGate6" H 5065 2946 50  0000 L CNN
+F 0 "CDrGate1" H 5065 2946 50  0000 L CNN
 F 1 "0.47uF" H 5065 2854 50  0000 L CNN
 F 2 "Capacitors_SMD:C_0603_HandSoldering" H 4988 2750 30  0001 C CNN
@@
 AR Path="/56BA2E2B/56984538" Ref="Usens5"  Part="1"
 AR Path="/56BA5F82/56984538" Ref="Usens6"  Part="1"
-F 0 "Usens6" V 7797 2922 60  0000 R CNN
+F 0 "Usens1" V 7797 2922 60  0000 R CNN
 F 1 "ACS711" V 7903 2922 60  0000 R CNN
 F 2 "Allegro:QFN-12-1EX_3x3mm_Pitch0.5mm" V 7956 2922 60  0001 R CNN
@@
 AR Path="/56BA2E2B/56A19C85" Ref="UDrmos5"  Part="1"
 AR Path="/56BA5F82/56A19C85" Ref="UDrmos6"  Part="1"
-F 0 "UDrmos6" H 5650 5071 50  0000 C CNN
+F 0 "UDrmos1" H 5650 5071 50  0000 C CNN
 F 1 "DrMOS_SiC632A" H 5650 4979 50  0000 C CNN
 F 2 "DrMOS:MLP55-31L" H 5650 4887 50  0000 C CNN
@@
 AR Path="/56BA2E2B/56A2CDC4" Ref="CDrLogic5"  Part="1"
 AR Path="/56BA5F82/56A2CDC4" Ref="CDrLogic6"  Part="1"
-F 0 "CDrLogic6" H 4415 3446 50  0000 L CNN
+F 0 "CDrLogic1" H 4415 3446 50  0000 L CNN
 F 1 "2.2uF" H 4415 3354 50  0000 L CNN
 F 2 "Capacitors_SMD:C_0603" H 4338 3250 30  0001 C CNN
@@
 AR Path="/56BA2E2B/56A2D0BC" Ref="RDrLogic5"  Part="1"
 AR Path="/56BA5F82/56A2D0BC" Ref="RDrLogic6"  Part="1"
-F 0 "RDrLogic6" H 4370 2946 50  0000 L CNN
+F 0 "RDrLogic1" H 4370 2946 50  0000 L CNN
 F 1 "R" H 4370 2854 50  0000 L CNN
 F 2 "Resistors_SMD:R_0603" V 4230 2900 50  0001 C CNN
@@
 AR Path="/56BA2E2B/56A2FD69" Ref="Rhsens5"  Part="1"
 AR Path="/56BA5F82/56A2FD69" Ref="Rhsens6"  Part="1"
-F 0 "Rhsens6" H 7520 4346 50  0000 L CNN
+F 0 "Rhsens1" H 7520 4346 50  0000 L CNN
 F 1 "10k" H 7520 4254 50  0000 L CNN
 F 2 "Capacitors_SMD:C_0603_HandSoldering" V 7380 4300 50  0001 C CNN
@@
 AR Path="/56BA2E2B/56A2FEAC" Ref="Rlsens5"  Part="1"
 AR Path="/56BA5F82/56A2FEAC" Ref="Rlsens6"  Part="1"
-F 0 "Rlsens6" H 7520 4746 50  0000 L CNN
+F 0 "Rlsens1" H 7520 4746 50  0000 L CNN
 F 1 "2k2" H 7520 4654 50  0000 L CNN
 F 2 "Resistors_SMD:R_0402" V 7380 4700 50  0001 C CNN
@@
 AR Path="/56BA2E2B/56A3225A" Ref="Rcfilt5"  Part="1"
 AR Path="/56BA5F82/56A3225A" Ref="Rcfilt6"  Part="1"
-F 0 "Rcfilt6" H 8420 2846 50  0000 L CNN
+F 0 "Rcfilt1" H 8420 2846 50  0000 L CNN
 F 1 "R" H 8420 2754 50  0000 L CNN
 F 2 "Resistors_SMD:R_0402" V 8280 2800 50  0001 C CNN
@@
 AR Path="/56BA2E2B/56A3233B" Ref="Ccfilt5"  Part="1"
 AR Path="/56BA5F82/56A3233B" Ref="Ccfilt6"  Part="1"
-F 0 "Ccfilt6" H 8165 2846 50  0000 L CNN
+F 0 "Ccfilt1" H 8165 2846 50  0000 L CNN
 F 1 "C" H 8165 2754 50  0000 L CNN
 F 2 "Capacitors_SMD:C_0402" H 8088 2650 50  0001 C CNN
@@
 AR Path="/56BA2E2B/56A69B0E" Ref="CDrHV5"  Part="1"
 AR Path="/56BA5F82/56A69B0E" Ref="CDrHV6"  Part="1"
-F 0 "CDrHV6" H 5865 1246 50  0000 L CNN
+F 0 "CDrHV1" H 5865 1246 50  0000 L CNN
 F 1 "10u" H 5865 1154 50  0000 L CNN
 F 2 "Capacitors_SMD:C_1206" H 5788 1050 50  0001 C CNN
@@
 AR Path="/56BA2E2B/56AF6D20" Ref="CDrHVs5"  Part="1"
 AR Path="/56BA5F82/56AF6D20" Ref="CDrHVs6"  Part="1"
-F 0 "CDrHVs6" H 5315 1246 50  0000 L CNN
+F 0 "CDrHVs1" H 5315 1246 50  0000 L CNN
 F 1 "0.47u" H 5315 1154 50  0000 L CNN
 F 2 "Capacitors_SMD:C_0603" H 5315 1108 50  0001 L CNN
@@
 AR Path="/56BA2E2B/56B30AD6" Ref="PMotor5"  Part="1"
 AR Path="/56BA5F82/56B30AD6" Ref="PMotor6"  Part="1"
-F 0 "PMotor6" H 9177 4106 60  0000 L CNN
+F 0 "PMotor1" H 9177 4106 60  0000 L CNN
 F 1 "PAD_SMD" H 9177 4000 60  0000 L CNN
 F 2 "CRF1:1PAD_4x5mm" H 9177 3894 60  0000 L CNN
@@
 AR Path="/56BA2E2B/56B897AB" Ref="Csens5"  Part="1"
 AR Path="/56BA5F82/56B897AB" Ref="Csens6"  Part="1"
-F 0 "Csens6" H 6965 2142 50  0000 L CNN
+F 0 "Csens1" H 6965 2142 50  0000 L CNN
 F 1 "0.47u" H 6965 2050 50  0000 L CNN
 F 2 "Capacitors_SMD:C_0603" H 6965 1958 50  0000 L CNN

Commit message: Added some part numbers for the BOM
Parts:
- CDrGate1, Csens1: Comment (none) -> X7R, >10V
- CDrLogic1: Comment (none) -> X7R, >10V; Manufacturer (none) -> Kemet; Part Number (none) -> C0603C225K8RACTU
- UDrmos1: Manufacturer (none) -> Vishay; Part Number (none) -> SiC632CD-T1-GE3
- Usens1: Manufacturer (none) -> Allegro; Part Number (none) -> ACS711KEXLT-31AB-T
Changed lines of the file:
@@
 $Descr A4 11693 8268
 encoding utf-8
-Sheet 4 11
+Sheet 3 11
 Title "DrMOS power stage"
 Date "2016-01-22"
@@
 AR Path="/56BA2E2B/55DF8D4F" Ref="Cboot5"  Part="1"
 AR Path="/56BA5F82/55DF8D4F" Ref="Cboot6"  Part="1"
-F 0 "Cboot6" V 6647 3700 50  0000 C CNN
+F 0 "Cboot1" V 6647 3700 50  0000 C CNN
 F 1 "0.47uF" V 6739 3700 50  0000 C CNN
 F 2 "Capacitors_SMD:C_0603_HandSoldering" H 6938 3550 30  0001 C CNN
@@
 AR Path="/56BA2E2B/55DF8D84" Ref="CDrGate5"  Part="1"
 AR Path="/56BA5F82/55DF8D84" Ref="CDrGate6"  Part="1"
-F 0 "CDrGate6" H 5065 2946 50  0000 L CNN
+F 0 "CDrGate1" H 5065 2946 50  0000 L CNN
 F 1 "0.47uF" H 5065 2854 50  0000 L CNN
 F 2 "Capacitors_SMD:C_0603_HandSoldering" H 4988 2750 30  0001 C CNN
 F 3 "" H 4950 2900 60  0000 C CNN
+F 4 "X7R, >10V" H 4950 2900 60  0001 C CNN "Comment"
 	1    4950 2900
 	1    0    0    -1
@@
 AR Path="/56BA2E2B/56984538" Ref="Usens5"  Part="1"
 AR Path="/56BA5F82/56984538" Ref="Usens6"  Part="1"
-F 0 "Usens6" V 7797 2922 60  0000 R CNN
+F 0 "Usens1" V 7797 2922 60  0000 R CNN
 F 1 "ACS711" V 7903 2922 60  0000 R CNN
 F 2 "Allegro:QFN-12-1EX_3x3mm_Pitch0.5mm" V 7956 2922 60  0001 R CNN
 F 3 "" H 7700 3750 60  0000 C CNN
+F 4 "Allegro" V 7850 3550 60  0001 C CNN "Manufacturer"
+F 5 "ACS711KEXLT-31AB-T" V 7850 3550 60  0001 C CNN "Part Number"
 	1    7850 3550
 	0    -1   1    0
@@
 AR Path="/56BA2E2B/56A19C85" Ref="UDrmos5"  Part="1"
 AR Path="/56BA5F82/56A19C85" Ref="UDrmos6"  Part="1"
-F 0 "UDrmos6" H 5650 5071 50  0000 C CNN
+F 0 "UDrmos1" H 5650 5071 50  0000 C CNN
 F 1 "DrMOS_SiC632A" H 5650 4979 50  0000 C CNN
 F 2 "DrMOS:MLP55-31L" H 5650 4887 50  0000 C CNN
 F 3 "" H 5850 3800 50  0000 C CNN
+F 4 "Vishay" H 5850 4000 60  0001 C CNN "Manufacturer"
+F 5 "SiC632CD-T1-GE3" H 5850 4000 60  0001 C CNN "Part Number"
 	1    5850 4000
 	1    0    0    -1
@@
 AR Path="/56BA2E2B/56A2AE4F" Ref="#PWR077"  Part="1"
 AR Path="/56BA5F82/56A2AE4F" Ref="#PWR090"  Part="1"
-F 0 "#PWR090" H 5750 4850 50  0001 C CNN
+F 0 "#PWR015" H 5750 4850 50  0001 C CNN
 F 1 "GNDPWR" H 5750 4900 50  0000 C CNN
 F 2 "" H 5750 5000 50  0000 C CNN
@@
 AR Path="/56BA2E2B/56A2B769" Ref="#PWR078"  Part="1"
 AR Path="/56BA5F82/56A2B769" Ref="#PWR091"  Part="1"
-F 0 "#PWR091" H 5200 4750 50  0001 C CNN
+F 0 "#PWR016" H 5200 4750 50  0001 C CNN
 F 1 "GND" H 5208 4826 50  0000 C CNN
 F 2 "" H 5200 5000 50  0000 C CNN
@@
 AR Path="/56BA2E2B/56A2BBEE" Ref="#PWR079"  Part="1"
 AR Path="/56BA5F82/56A2BBEE" Ref="#PWR092"  Part="1"
-F 0 "#PWR092" H 4950 3000 50  0001 C CNN
+F 0 "#PWR017" H 4950 3000 50  0001 C CNN
 F 1 "GNDPWR" H 4957 3275 50  0000 C CNN
 F 2 "" H 4950 3150 50  0000 C CNN
@@
 AR Path="/56BA2E2B/56A2CDC4" Ref="CDrLogic5"  Part="1"
 AR Path="/56BA5F82/56A2CDC4" Ref="CDrLogic6"  Part="1"
-F 0 "CDrLogic6" H 4415 3446 50  0000 L CNN
+F 0 "CDrLogic1" H 4415 3446 50  0000 L CNN
 F 1 "2.2uF" H 4415 3354 50  0000 L CNN
 F 2 "Capacitors_SMD:C_0603" H 4338 3250 30  0001 C CNN
 F 3 "" H 4300 3400 60  0000 C CNN
+F 4 "Kemet" H 4300 3400 60  0001 C CNN "Manufacturer"
+F 5 "C0603C225K8RACTU" H 4300 3400 60  0001 C CNN "Part Number"
+F 6 "X7R, >10V" H 4300 3400 60  0001 C CNN "Comment"
 	1    4300 3400
 	1    0    0    -1
@@
 AR Path="/56BA2E2B/56A2CDEC" Ref="#PWR080"  Part="1"
 AR Path="/56BA5F82/56A2CDEC" Ref="#PWR093"  Part="1"
-F 0 "#PWR093" H 4300 3300 50  0001 C CNN
+F 0 "#PWR018" H 4300 3300 50  0001 C CNN
 F 1 "GND" H 4308 3376 50  0000 C CNN
 F 2 "" H 4300 3550 50  0000 C CNN
@@
 AR Path="/56BA2E2B/56A2CF9B" Ref="#PWR081"  Part="1"
 AR Path="/56BA5F82/56A2CF9B" Ref="#PWR094"  Part="1"
-F 0 "#PWR094" H 4300 2500 50  0001 C CNN
+F 0 "#PWR019" H 4300 2500 50  0001 C CNN
 F 1 "+5V" H 4318 2824 50  0000 C CNN
 F 2 "" H 4300 2650 50  0000 C CNN
@@
 AR Path="/56BA2E2B/56A2D0BC" Ref="RDrLogic5"  Part="1"
 AR Path="/56BA5F82/56A2D0BC" Ref="RDrLogic6"  Part="1"
-F 0 "RDrLogic6" H 4370 2946 50  0000 L CNN
+F 0 "RDrLogic1" H 4370 2946 50  0000 L CNN
 F 1 "R" H 4370 2854 50  0000 L CNN
 F 2 "Resistors_SMD:R_0603" V 4230 2900 50  0001 C CNN
@@
 AR Path="/56BA2E2B/56A2EFF6" Ref="#PWR082"  Part="1"
 AR Path="/56BA5F82/56A2EFF6" Ref="#PWR095"  Part="1"
-F 0 "#PWR095" H 8550 2800 50  0001 C CNN
+F 0 "#PWR020" H 8550 2800 50  0001 C CNN
 F 1 "GND" H 8558 2876 50  0000 C CNN
 F 2 "" H 8550 3050 50  0000 C CNN
@@
 AR Path="/56BA2E2B/56A2FD69" Ref="Rhsens5"  Part="1"
 AR Path="/56BA5F82/56A2FD69" Ref="Rhsens6"  Part="1"
-F 0 "Rhsens6" H 7520 4346 50  0000 L CNN
+F 0 "Rhsens1" H 7520 4346 50  0000 L CNN
 F 1 "10k" H 7520 4254 50  0000 L CNN
 F 2 "Capacitors_SMD:C_0603_HandSoldering" V 7380 4300 50  0001 C CNN
@@
 AR Path="/56BA2E2B/56A2FEAC" Ref="Rlsens5"  Part="1"
 AR Path="/56BA5F82/56A2FEAC" Ref="Rlsens6"  Part="1"
-F 0 "Rlsens6" H 7520 4746 50  0000 L CNN
+F 0 "Rlsens1" H 7520 4746 50  0000 L CNN
 F 1 "2k2" H 7520 4654 50  0000 L CNN
 F 2 "Resistors_SMD:R_0402" V 7380 4700 50  0001 C CNN
@@
 AR Path="/56BA2E2B/56A30067" Ref="#PWR083"  Part="1"
 AR Path="/56BA5F82/56A30067" Ref="#PWR096"  Part="1"
-F 0 "#PWR096" H 7450 4700 50  0001 C CNN
+F 0 "#PWR021" H 7450 4700 50  0001 C CNN
 F 1 "GND" H 7458 4776 50  0000 C CNN
 F 2 "" H 7450 4950 50  0000 C CNN
@@
 AR Path="/56BA2E2B/56A31D68" Ref="#PWR084"  Part="1"
 AR Path="/56BA5F82/56A31D68" Ref="#PWR097"  Part="1"
-F 0 "#PWR097" H 6050 2850 50  0001 C CNN
+F 0 "#PWR022" H 6050 2850 50  0001 C CNN
 F 1 "+24V" H 6068 3174 50  0000 C CNN
 F 2 "" H 6050 3000 50  0000 C CNN
@@
 AR Path="/56BA2E2B/56A32138" Ref="#PWR085"  Part="1"
 AR Path="/56BA5F82/56A32138" Ref="#PWR098"  Part="1"
-F 0 "#PWR098" H 7350 2500 50  0001 C CNN
+F 0 "#PWR023" H 7350 2500 50  0001 C CNN
 F 1 "+3.3V" H 7368 2824 50  0000 C CNN
 F 2 "" H 7350 2650 50  0000 C CNN
@@
 AR Path="/56BA2E2B/56A3225A" Ref="Rcfilt5"  Part="1"
 AR Path="/56BA5F82/56A3225A" Ref="Rcfilt6"  Part="1"
-F 0 "Rcfilt6" H 8420 2846 50  0000 L CNN
+F 0 "Rcfilt1" H 8420 2846 50  0000 L CNN
 F 1 "R" H 8420 2754 50  0000 L CNN
 F 2 "Resistors_SMD:R_0402" V 8280 2800 50  0001 C CNN
@@
 AR Path="/56BA2E2B/56A3233B" Ref="Ccfilt5"  Part="1"
 AR Path="/56BA5F82/56A3233B" Ref="Ccfilt6"  Part="1"
-F 0 "Ccfilt6" H 8165 2846 50  0000 L CNN
+F 0 "Ccfilt1" H 8165 2846 50  0000 L CNN
 F 1 "C" H 8165 2754 50  0000 L CNN
 F 2 "Capacitors_SMD:C_0402" H 8088 2650 50  0001 C CNN
@@
 AR Path="/56BA2E2B/56A69AD2" Ref="#PWR086"  Part="1"
 AR Path="/56BA5F82/56A69AD2" Ref="#PWR099"  Part="1"
-F 0 "#PWR099" H 5750 800 50  0001 C CNN
+F 0 "#PWR024" H 5750 800 50  0001 C CNN
 F 1 "+24V" H 5768 1124 50  0000 C CNN
 F 2 "" H 5750 950 50  0000 C CNN
@@
 AR Path="/56BA2E2B/56A69B0E" Ref="CDrHV5"  Part="1"
 AR Path="/56BA5F82/56A69B0E" Ref="CDrHV6"  Part="1"
-F 0 "CDrHV6" H 5865 1246 50  0000 L CNN
+F 0 "CDrHV1" H 5865 1246 50  0000 L CNN
 F 1 "10u" H 5865 1154 50  0000 L CNN
 F 2 "Capacitors_SMD:C_1206" H 5788 1050 50  0001 C CNN
@@
 AR Path="/56BA2E2B/56A69BA7" Ref="#PWR087"  Part="1"
 AR Path="/56BA5F82/56A69BA7" Ref="#PWR0100"  Part="1"
-F 0 "#PWR0100" H 5750 1300 50  0001 C CNN
+F 0 "#PWR025" H 5750 1300 50  0001 C CNN
 F 1 "GNDPWR" H 5757 1575 50  0000 C CNN
 F 2 "" H 5750 1450 50  0000 C CNN
@@
 AR Path="/56BA2E2B/56AF6D20" Ref="CDrHVs5"  Part="1"
 AR Path="/56BA5F82/56AF6D20" Ref="CDrHVs6"  Part="1"
-F 0 "CDrHVs6" H 5315 1246 50  0000 L CNN
+F 0 "CDrHVs1" H 5315 1246 50  0000 L CNN
 F 1 "0.47u" H 5315 1154 50  0000 L CNN
 F 2 "Capacitors_SMD:C_0603" H 5315 1108 50  0001 L CNN
@@
 AR Path="/56BA2E2B/56B30AD6" Ref="PMotor5"  Part="1"
 AR Path="/56BA5F82/56B30AD6" Ref="PMotor6"  Part="1"
-F 0 "PMotor6" H 9177 4106 60  0000 L CNN
+F 0 "PMotor1" H 9177 4106 60  0000 L CNN
 F 1 "PAD_SMD" H 9177 4000 60  0000 L CNN
 F 2 "CRF1:1PAD_4x5mm" H 9177 3894 60  0000 L CNN
@@
 AR Path="/56BA2E2B/56B897AB" Ref="Csens5"  Part="1"
 AR Path="/56BA5F82/56B897AB" Ref="Csens6"  Part="1"
-F 0 "Csens6" H 6965 2142 50  0000 L CNN
+F 0 "Csens1" H 6965 2142 50  0000 L CNN
 F 1 "0.47u" H 6965 2050 50  0000 L CNN
 F 2 "Capacitors_SMD:C_0603" H 6965 1958 50  0000 L CNN
 F 3 "" H 6850 2050 50  0000 C CNN
+F 4 "X7R, >10V" H 6850 2050 60  0001 C CNN "Comment"
 	1    6850 2050
 	1    0    0    -1
@@
 AR Path="/56BA2E2B/56B89931" Ref="#PWR088"  Part="1"
 AR Path="/56BA5F82/56B89931" Ref="#PWR0101"  Part="1"
-F 0 "#PWR0101" H 6850 1950 50  0001 C CNN
+F 0 "#PWR026" H 6850 1950 50  0001 C CNN
 F 1 "GND" H 6858 2026 50  0000 C CNN
 F 2 "" H 6850 2200 50  0000 C CNN
@@
 AR Path="/56BA2E2B/56B89961" Ref="#PWR089"  Part="1"
 AR Path="/56BA5F82/56B89961" Ref="#PWR0102"  Part="1"
-F 0 "#PWR0102" H 6850 1750 50  0001 C CNN
+F 0 "#PWR027" H 6850 1750 50  0001 C CNN
 F 1 "+3.3V" H 6868 2074 50  0000 C CNN
 F 2 "" H 6850 1900 50  0000 C CNN
