File: hardware/design/STM32F4 64LQFP.sch (KiCad schematic (older format))
At the start: 16 parts, among them U1 STM32F40X_LQFP64, X2 8MHz 10ppm

Commit message: Added pullup resistor for THWn. Fixed some not connected parts warnings.
Parts:
- added Rthwn1: 2k7, Resistors_SMD:R_0402, symbol R
- R3: value R/DNP -> 2k7/DNP
Connections:
- net +3V3: now also Rthwn1.1
- net THWn: now also Rthwn1.2
Other:
- note added: "Muss hin!"
Changed lines of the file:
@@
 P 7200 2550
 F 0 "R3" V 6992 2550 50  0000 C CNN
-F 1 "R/DNP" V 7084 2550 50  0000 C CNN
+F 1 "2k7/DNP" V 7084 2550 50  0000 C CNN
 F 2 "Resistors_SMD:R_0402" V 7084 2550 50  0001 C CNN
 F 3 "" H 7200 2550 50  0000 C CNN
@@
 Wire Wire Line
 	9100 1600 10150 1600
+$Comp
+L R Rthwn1
+U 1 1 577AD1BD
+P 8600 2200
+F 0 "Rthwn1" H 8670 2292 50  0000 L CNN
+F 1 "2k7" H 8670 2200 50  0000 L CNN
+F 2 "Resistors_SMD:R_0402" H 8670 2108 50  0000 L CNN
+F 3 "" H 8600 2200 50  0000 C CNN
+	1    8600 2200
+	1    0    0    -1
+$EndComp
+$Comp
+L +3.3V #PWR0114
+U 1 1 577AD239
+P 8600 2050
+F 0 "#PWR0114" H 8600 1900 50  0001 C CNN
+F 1 "+3.3V" H 8618 2224 50  0000 C CNN
+F 2 "" H 8600 2050 50  0000 C CNN
+F 3 "" H 8600 2050 50  0000 C CNN
+	1    8600 2050
+	1    0    0    -1
+$EndComp
+Wire Wire Line
+	8600 2350 8600 2450
+Connection ~ 8600 2450
+Text Notes 7400 2450 0    60   ~ 0
+Muss hin!
 $EndSCHEMATC

Commit message: Fixed Crystal pin 4 not connected to GND
Parts:
- X2: footprint CRF1:Crystal_5x3mm -> Crystals_User:Crystal_5x3mm
Changed lines of the file:
@@
 F 0 "X2" H 7750 2225 30  0000 C CNN
 F 1 "8MHz 10ppm" H 7750 2164 30  0000 C CNN
-F 2 "CRF1:Crystal_5x3mm" H 7750 2050 60  0001 C CNN
+F 2 "Crystals_User:Crystal_5x3mm" H 7750 2050 60  0001 C CNN
 F 3 "" H 7750 2050 60  0000 C CNN
 F 4 "ABM3B-8.0-10-1UT" H 7750 2050 60  0001 C CNN "mfg#"
