File: hardware/design/virtual_y.sch (KiCad schematic (older format))
At the start: 13 parts

Commit message: TODO Double-check BOM. Check silk screen. Check Gerber output.
Parts:
- CHFAC1: value C -> 10n; Comment (none) -> Use COG or NPO ceramic. Or poly- propylene or carbonate
- Dclamp1: Manufacturer (none) -> NXP; Part Number (none) -> BAT754S
- RHFAC1: value R -> 100R
- RYOFFS1: value R -> 20k
- RYSGND1: value 0R/DNP -> 20k
Changed lines of the file:
@@
 P 4650 5850
 F 0 "RYSGND1" V 4443 5850 50  0000 C CNN
-F 1 "0R/DNP" V 4534 5850 50  0000 C CNN
+F 1 "20k" V 4534 5850 50  0000 C CNN
 F 2 "Resistors_SMD:R_0402" V 4580 5850 50  0001 C CNN
 F 3 "" H 4650 5850 50  0000 C CNN
@@
 P 5350 5650
 F 0 "RHFAC1" V 5143 5650 50  0000 C CNN
-F 1 "R" V 5234 5650 50  0000 C CNN
+F 1 "100R" V 5234 5650 50  0000 C CNN
 F 2 "Resistors_SMD:R_0603_HandSoldering" V 5280 5650 50  0001 C CNN
 F 3 "" H 5350 5650 50  0000 C CNN
@@
 P 5800 5650
 F 0 "CHFAC1" V 5548 5650 50  0000 C CNN
-F 1 "C" V 5639 5650 50  0000 C CNN
+F 1 "10n" V 5639 5650 50  0000 C CNN
 F 2 "Capacitors_SMD:C_0603_HandSoldering" H 5838 5500 50  0001 C CNN
 F 3 "" H 5800 5650 50  0000 C CNN
+F 4 "Use COG or NPO ceramic. Or poly- propylene or carbonate" V 5800 5650 60  0001 C CNN "Comment"
 	1    5800 5650
 	0    1    1    0
@@
 P 4650 5350
 F 0 "RYOFFS1" H 4720 5396 50  0000 L CNN
-F 1 "R" H 4720 5305 50  0000 L CNN
+F 1 "20k" H 4720 5305 50  0000 L CNN
 F 2 "Resistors_SMD:R_0603_HandSoldering" V 4580 5350 50  0001 C CNN
 F 3 "" H 4650 5350 50  0000 C CNN
@@
 F 2 "TO_SOT_Packages_SMD:SOT-23" H 4300 5650 50  0001 C CNN
 F 3 "" H 4300 5650 50  0000 C CNN
+F 4 "NXP" V 4300 5650 60  0001 C CNN "Manufacturer"
+F 5 "BAT754S" V 4300 5650 60  0001 C CNN "Part Number"
 	1    4300 5650
 	0    -1   -1   0

Commit message: Added just a few words...
Parts:
- CHFAC1: value 10n -> 10n,35V
Changed lines of the file:
@@
 encoding utf-8
 Sheet 5 11
-Title ""
+Title "Alternate voltage sensing options"
 Date ""
 Rev "0.1"
@@
 P 5800 5650
 F 0 "CHFAC1" V 5548 5650 50  0000 C CNN
-F 1 "10n" V 5639 5650 50  0000 C CNN
+F 1 "10n,35V" V 5639 5650 50  0000 C CNN
 F 2 "Capacitors_SMD:C_0603_HandSoldering" H 5838 5500 50  0001 C CNN
 F 3 "" H 5800 5650 50  0000 C CNN
@@
 Wire Wire Line
 	5950 5650 6050 5650
-Text Notes 6900 5100 0    60   ~ 0
+Text Notes 5100 6250 0    60   ~ 0
 PHFAC - High Frequency AC sensing on SENSY2\n- voltage divider RYSGND/(RYOFFS+RYSGND) sets the offset for SENSY2\n- the gain is set by RHFAC/(RHFAC+RYOFFS||RYSGND)\n- DZLIM limits the ADC input to 3.3V
 $Comp
